File: Esp32-C3-02.kicad_sch (KiCad schematic)
At the start: 30 parts, among them J3 GSD090012SEU, U2 USBLC6-2SC6, U3 ESP32-C3-WROOM-02, U4 CP2102N-Axx-xQFN20, U5 W25Q16JVSS

Commit message: assigning footprint, pcb setup and configurations
Parts:
- C12, C7, C9: footprint Capacitor_Tantalum_SMD:CP_EIA-7343-40_Kemet-Y -> FootPrints:CAPMP3216X180N
- J3: footprint GSD090012SEU:AMPHENOL_GSD090012SEU -> FootPrints:AMPHENOL_GSD090012SEU
- U4: footprint Package_DFN_QFN:SiliconLabs_QFN-20-1EP_3x3mm_P0.5mm -> FootPrints:WFQFN-20
Changed lines of the file:
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@@
 			)
 		)
-		(property "Footprint" "Capacitor_Tantalum_SMD:CP_EIA-7343-40_Kemet-Y"
+		(property "Footprint" "FootPrints:CAPMP3216X180N"
 			(at 63.881 29.5148 0)
 			(effects
@@
 			)
 		)
-		(property "Footprint" "Package_DFN_QFN:SiliconLabs_QFN-20-1EP_3x3mm_P0.5mm"
+		(property "Footprint" "FootPrints:WFQFN-20"
 			(at 124.206 100.965 0)
 			(effects
@@
 			)
 		)
-		(property "Footprint" "Capacitor_Tantalum_SMD:CP_EIA-7343-40_Kemet-Y"
+		(property "Footprint" "FootPrints:CAPMP3216X180N"
 			(at 263.8552 72.39 0)
 			(effects
@@
 			)
 		)
-		(property "Footprint" "GSD090012SEU:AMPHENOL_GSD090012SEU"
+		(property "Footprint" "FootPrints:AMPHENOL_GSD090012SEU"
 			(at 46.228 155.956 0)
 			(effects
@@
 			)
 		)
-		(property "Footprint" "Capacitor_Tantalum_SMD:CP_EIA-7343-40_Kemet-Y"
+		(property "Footprint" "FootPrints:CAPMP3216X180N"
 			(at 100.3808 164.338 0)
 			(effects
