File: user_interface.kicad_sch (KiCad schematic)
At the start: 0 parts

Commit message: initial commit user-interface schematic
Parts:
- added J4: Conn_01x04_Pin, symbol Connector:Conn_01x04_Pin
- added J5: Conn_01x05_Pin, symbol Connector:Conn_01x05_Pin
- added S1, S2: USLPT2819DT2TR, USLPT2819DT2TR:SW_USLPT2819DT2TR, symbol USLPT2819DT2TR:USLPT2819DT2TR
Connections:
- new net +3.3V: J4.1 (Pin_1), J5.1 (Pin_1)
- new net GND: J4.4 (Pin_4), J5.5 (Pin_5)
- new net GPIO18: J5.3 (Pin_3)
- new net GPIO19: J5.4 (Pin_4)
- new net GPIO8: J5.2 (Pin_2)
- new net SCL: J4.2 (Pin_2)
- new net SDA: J4.3 (Pin_3)
Other:
- note added: "BreakOut for Remaining Pins"
- note added: "OLED DISPLAY"

Commit message: final touch on user interface schematic
Parts:
- added C21: 0.1u, symbol Device:C
- added C22: 1u, symbol Device:C
- added Q2, Q3: BC817, Package_TO_SOT_SMD:SOT-23, symbol Transistor_BJT:BC817
- added R32, R33, R34: 10K, symbol Device:R
Connections:
- net +3.3V: now also R32.1
- net GND: now also S1.1, S1.2, S2.1, S2.2, C21.2, C22.2
- net BOOT: now reaches S1.3
- net BOOT: now also S1.4, C21.1, Q3.2 (E)
- net EN: now reaches S2.3
- net EN: now also S2.4, C22.1, Q2.3 (C), R32.2
- new net: Q2.1 (B), R33.2
- new net: Q3.1 (B), R34.2
- new net DTR: Q3.3 (C), R33.1
- new net RTS: Q2.2 (E), R34.1
Other:
- note added: "AUTO Program DTR RTS -> EN I00 I02 1 1 1 1 1 0 0 1 1 1 1 0 0 1 1 0 1 1 0 0"
- note added: "BOOT"
- note added: "RESET"
- note added: "To learn more about the ESP32 boot mode got to texplo.re/esp32boot"

Commit message: run ERC check for the schematic
Parts:
- C21, C22: footprint (none) -> Capacitor_SMD:C_0805_2012Metric
- J4: footprint (none) -> Connector_PinHeader_2.54mm:PinHeader_1x04_P2.54mm_Vertical
- J5: footprint (none) -> Connector_PinHeader_2.54mm:PinHeader_1x05_P2.54mm_Vertical
- R32, R33, R34: footprint (none) -> Resistor_SMD:R_0805_2012Metric
Changed lines of the file:
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@@
 			)
 		)
-		(property "Footprint" ""
+		(property "Footprint" "Capacitor_SMD:C_0805_2012Metric"
 			(at 132.7912 68.58 0)
 			(effects
@@
 			)
 		)
-		(property "Footprint" ""
+		(property "Footprint" "Capacitor_SMD:C_0805_2012Metric"
 			(at 196.0372 68.072 0)
 			(effects
@@
 			)
 		)
-		(property "Footprint" ""
+		(property "Footprint" "Resistor_SMD:R_0805_2012Metric"
 			(at 154.94 115.57 90)
 			(effects
@@
 			)
 		)
-		(property "Footprint" ""
+		(property "Footprint" "Connector_PinHeader_2.54mm:PinHeader_1x05_P2.54mm_Vertical"
 			(at 43.688 82.55 0)
 			(effects
@@
 			)
 		)
-		(property "Footprint" ""
+		(property "Footprint" "Resistor_SMD:R_0805_2012Metric"
 			(at 155.448 131.318 90)
 			(effects
@@
 			)
 		)
-		(property "Footprint" ""
+		(property "Footprint" "Resistor_SMD:R_0805_2012Metric"
 			(at 185.928 45.974 90)
 			(effects
@@
 			)
 		)
-		(property "Footprint" ""
+		(property "Footprint" "Connector_PinHeader_2.54mm:PinHeader_1x04_P2.54mm_Vertical"
 			(at 38.354 39.116 0)
 			(effects

Commit message: assigning footprint, pcb setup and configurations
Parts:
- S1, S2: footprint USLPT2819DT2TR:SW_USLPT2819DT2TR -> FootPrints:SW_USLPT2819DT2TR
Changed lines of the file:
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@@
 			)
 		)
-		(property "Footprint" "USLPT2819DT2TR:SW_USLPT2819DT2TR"
+		(property "Footprint" "FootPrints:SW_USLPT2819DT2TR"
 			(at 146.304 50.8 0)
 			(effects
@@
 			)
 		)
-		(property "Footprint" "USLPT2819DT2TR:SW_USLPT2819DT2TR"
+		(property "Footprint" "FootPrints:SW_USLPT2819DT2TR"
 			(at 208.28 50.8 0)
 			(effects
